Commit message: add URDF joint limit

File: description/urdf/my_robot.description.urdf.xacro (robot description, xacro)
@@ -19,5 +19,5 @@
   <material name="robot_yellow">
     <color rgba="0.9 0.9 0.1 1"/>
-  </material>
+    </material>
   <material name="robot_orange">
     <color rgba="1.0 0.5 0.1 1"/>
@@ -28,8 +28,6 @@
   <!-- Xacro properties for common values -->
   <xacro:property name="mesh_scale" value="0.001 0.001 0.001"/>
-  <xacro:property name="joint_effort" value="0.0"/>
-  <xacro:property name="joint_velocity" value="0.0"/>
-  <xacro:property name="joint_lower_limit" value="-3.14"/>
-  <xacro:property name="joint_upper_limit" value="3.14"/>
+  <!-- Define pi for use in expressions -->
+  <xacro:property name="pi" value="3.14159265359"/>
   <!-- Macro for mesh link -->
   <xacro:macro name="mesh_link" params="name mesh_file material_name collision_xyz:='0 0 0' visual_xyz:='0 0 0' collision_geometry:=''">
@@ -44,5 +42,5 @@
             <box size="0.07 0.115 0.015"/>
           </xacro:if>
-          <!-- 필요시 다른 geometry 타입들 추가 -->
+          <!-- Add other geometry types as needed -->
         </geometry>
       </collision>
@@ -57,7 +55,7 @@
   </xacro:macro>
   <!-- Macro for revolute joint -->
-  <xacro:macro name="revolute_joint" params="name parent child xyz rpy axis">
+  <xacro:macro name="revolute_joint" params="name parent child xyz rpy axis lower upper velocity effort">
     <joint name="${name}" type="revolute">
-      <limit lower="${joint_lower_limit}" upper="${joint_upper_limit}" effort="${joint_effort}" velocity="${joint_velocity}"/>
+      <limit lower="${lower}" upper="${upper}" effort="${effort}" velocity="${velocity}"/>
       <origin rpy="${rpy}" xyz="${xyz}"/>
       <parent link="${parent}"/>
@@ -105,5 +103,9 @@
                         xyz="0 0 0.0507"
                         rpy="0 0 0"
-                        axis="0 0 1"/>
+                        axis="0 0 1"
+                        lower="${-7.0 * pi / 6.0}"
+                        upper="${pi / 6.0}"
+                        velocity="${23.0 * 2.0 * pi / 60.0}"
+                        effort="0.0"/>
   <xacro:mesh_link name="link1_1"
                    mesh_file="mesh_link1_1.stl"
@@ -140,5 +142,9 @@
                         xyz="0.009 0 0"
                         rpy="0 0 0"
-                        axis="1 0 0"/>
+                        axis="1 0 0"
+                        lower="${-pi / 2.0}"
+                        upper="${pi / 2.0}"
+                        velocity="${23.0 * 2.0 * pi / 60.0}"
+                        effort="0.0"/>
   <xacro:mesh_link name="link2_1"
                    mesh_file="mesh_link2_1.stl"
@@ -185,5 +191,9 @@
                         xyz="0 0 0.03905"
                         rpy="0 0 0"
-                        axis="0 0 1"/>
+                        axis="0 0 1"
+                        lower="${-23.0 * pi / 18.0}"
+                        upper="${pi / 3.0}"
+                        velocity="${148.0 * 2.0 * pi / 60.0}"
+                        effort="0.0"/>
   <xacro:mesh_link name="link3_1"
                    mesh_file="mesh_link3_1.stl"
@@ -219,5 +229,9 @@
                         xyz="-0.0065 0 0"
                         rpy="0 0 0"
-                        axis="-1 0 0"/>
+                        axis="-1 0 0"
+                        lower="${-19.0 * pi / 36.0}"
+                        upper="${19.0 * pi / 36.0}"
+                        velocity="${148.0 * 2.0 * pi / 60.0}"
+                        effort="0.0"/>
   <xacro:mesh_link name="link4_1"
                    mesh_file="mesh_link4_1.stl"
@@ -264,5 +278,9 @@
                         xyz="0 0 0.029"
                         rpy="0 0 0"
-                        axis="0 0 1"/>
+                        axis="0 0 1"
+                        lower="${-10.0 * pi / 9.0}"
+                        upper="${2.0 * pi / 3.0}"
+                        velocity="${233.0 * 2.0 * pi / 60.0}"
+                        effort="0.0"/>
   <xacro:mesh_link name="link5_1"
                    mesh_file="mesh_link5_1.stl"
@@ -298,5 +316,9 @@
                         xyz="0.002 0 0"
                         rpy="0 0 0"
-                        axis="1 0 0"/>
+                        axis="1 0 0"
+                        lower="${-19.0 * pi / 36.0}"
+                        upper="${19.0 * pi / 36.0}"
+                        velocity="${233.0 * 2.0 * pi / 60.0}"
+                        effort="0.0"/>
   <xacro:mesh_link name="link6_1"
                    mesh_file="mesh_link6_1.stl"
