Commit message: 조인트 리밋 추가 등

File: description/ros2_control/ros2_control_my_robot.xacro (robot description, xacro)
@@ -9,4 +9,6 @@
             <command_interface name="position"/>
             <state_interface name="position"/>
+            <param name="min">${-7.0 * pi / 6.0}</param>
+            <param name="max">${pi / 6.0}</param>
         </joint>
         <!-- Joint 2: Shoulder pitch (X-axis) -->
@@ -14,4 +16,6 @@
             <command_interface name="position"/>
             <state_interface name="position"/>
+            <param name="min">${-pi / 2.0}</param>
+            <param name="max">${pi / 2.0}</param>
         </joint>
         <!-- Joint 3: Elbow rotation (Z-axis) -->
@@ -19,4 +23,6 @@
             <command_interface name="position"/>
             <state_interface name="position"/>
+            <param name="min">${-23.0 * pi / 18.0}</param>
+            <param name="max">${pi / 3.0}</param>
         </joint>
         <!-- Joint 4: Wrist pitch (X-axis) -->
@@ -24,4 +30,6 @@
             <command_interface name="position"/>
             <state_interface name="position"/>
+            <param name="min">${-19.0 * pi / 36.0}</param>
+            <param name="max">${19.0 * pi / 36.0}</param>
         </joint>
         <!-- Joint 5: Wrist rotation (Z-axis) -->
@@ -29,4 +37,6 @@
             <command_interface name="position"/>
             <state_interface name="position"/>
+            <param name="min">${-10.0 * pi / 9.0}</param>
+            <param name="max">${2.0 * pi / 3.0}</param>
         </joint>
         <!-- Joint 6: End effector rotation (X-axis) -->
@@ -34,4 +44,6 @@
             <command_interface name="position"/>
             <state_interface name="position"/>
+            <param name="min">${-19.0 * pi / 36.0}</param>
+            <param name="max">${19.0 * pi / 36.0}</param>
         </joint>
     </ros2_control>

File: description/urdf/my_robot.description.urdf.xacro (robot description, xacro)
@@ -28,6 +28,4 @@
   <!-- Xacro properties for common values -->
   <xacro:property name="mesh_scale" value="0.001 0.001 0.001"/>
-  <!-- Define pi for use in expressions -->
-  <xacro:property name="pi" value="3.14159265359"/>
   <!-- Macro for mesh link -->
   <xacro:macro name="mesh_link" params="name mesh_file material_name collision_xyz:='0 0 0' visual_xyz:='0 0 0' collision_geometry:=''">
